File: Hardware/atmega32u4.sch (KiCad schematic (older format))
At the start: 1 part

Commit message: version 1 board completed
Parts:
- added C20, C27: 10uf, symbol CP1
- added C21, C22, C24: 0.1uf, symbol C
- added C23: 1uf, symbol C
- added C25, C26: 20pf, symbol C
- added CON1: USB-MINI-B, symbol USB-MINI-B
- added D1: Power LED, symbol LED
- added D2: DIODE, symbol DIODE
- added F8: FUSE, symbol FUSE
- added JP6: JUMPER, symbol JUMPER
- added P6, P7: CONN_01X12, symbol CONN_01X12
- added P8: CONN_02X03, symbol CONN_02X03
- added P9: CONN_01X06, symbol CONN_01X06
- added R14: 22, RES0603, symbol R
- added R15: 22, SM0603, symbol R
- added R16: 10k, RES0603, symbol R
- added R17: 1M, RES0603, symbol R
- added R18: 1k, RES0603, symbol R
- added SW1: SW_PUSH, symbol SW_PUSH
- added U3: MIC5329, ~, symbol MIC5329
- added X1: 16MHz, symbol CRYSTAL_SMD
- gave numbers to parts that had none: 1
Connections:
- net labels added: +5V, +BATT, 3.3V, 5V, A0, A1, A2, A3, A4, A5, ALERT_H, AREF, CONV_H, CS_H, D0/RX, D1/TX, D2/SDA, D3/SCL, D4, D5*, D6, D7, DRDY_H, FAULT_H, GND, HWB, IO10*, IO11*, IO12, IO13*, IO8, IO9*, MISO, MOSI, RST, RXLED, SCK, SCLK_H, SDI_H, SDO_H, TXLED, UCAP, USBID, VBUS, VCC
- wire segments 0 -> 148
- no-connect marks 0 -> 1
